File: fmc/hpc_example.brd (EAGLE design)
At the start: 160 x 100 mm, 4 parts

Commit message: added fmc lpc connector
updated naming
Parts:
- U$1: value FMC_HPC_M -> APS_HPC_M
- U$3: value FMC_HPC_F -> APS_HPC_F
Changed lines of the file:
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@@
 </autorouter>
 <elements>
-<element name="U$1" library="flipbit_fmc" package="ASP-134488-01" value="FMC_HPC_M" x="116.84" y="26.67"/>
+<element name="U$1" library="flipbit_fmc" package="ASP-134488-01" value="APS_HPC_M" x="116.84" y="26.67"/>
 <element name="U$2" library="flipbit_fmc" package="XILINX_FMC_MOUNT_CS" value="XILINX_FMC_MOUNT_CS" x="40.64" y="52.07"/>
-<element name="U$3" library="flipbit_fmc" package="ASP-134486-01" value="FMC_HPC_F" x="40.64" y="26.67"/>
+<element name="U$3" library="flipbit_fmc" package="ASP-134486-01" value="APS_HPC_F" x="40.64" y="26.67"/>
 <element name="U$4" library="flipbit_fmc" package="XILINX_FMC_MOUNT_BS" value="XILINX_FMC_MOUNT_BS" x="116.84" y="52.07"/>
 </elements>
